File: hw/boards/mta1-usb-v1/usb_to_serial.kicad_sch (KiCad schematic)
At the start: 10 parts, among them P1 USB_C_Plug, U3 CH552E, U5 USBLC6-2SC6

Commit message: Add extended values, manufacturer/distributor info to components in mta1
Parts:
- C13, C7: value 0.10uF -> (none); footprint mta1:CAPC1005X06L -> (none); Extended Value (none) -> 16V,X5R,20%; Manufacturer (none) -> Any/not critical
- P1: value USB_C_Plug -> (none); footprint mta1:U261-241N-4BS60 -> (none); Manufacturer (none) -> XKB; Manufacturer Part Number (none) -> U261-241N-4BS60; Supplier (none) -> LCSC; Supplier Part Number (none) -> C319150
- R29: value 5.1K -> (none); footprint mta1:ERJ2G(0402)_L -> (none); Extended Value (none) -> 1/16W,1%; Manufacturer (none) -> Any/not critical
- TP6, TP7, TP8, TP9: value INT_ICE_SCK -> (none); footprint TestPoint:TestPoint_Pad_D1.0mm -> (none); now left out of the parts list
- U3: value CH552E -> (none); footprint Package_SO:MSOP-10_3x3mm_P0.5mm -> (none); Manufacturer (none) -> WCH; Manufacturer Part Number (none) -> CH552E; Supplier (none) -> LCSC; Supplier Part Number (none) -> C967938
- U5: value USBLC6-2SC6 -> (none); footprint Package_TO_SOT_SMD:SOT-23-6 -> (none); Manufacturer (none) -> ST; Manufacturer Part Number (none) -> USBLC6-2SC6; Supplier (none) -> Digikey; Supplier Part Number (none) -> 497-5235-1-ND
Changed lines of the file:
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@@
       (effects (font (size 1.27 1.27)) (justify left))
     )
-    (property "Value" "USBLC6-2SC6" (id 1) (at 262.7376 114.173 90)
-      (effects (font (size 1.27 1.27)) (justify left))
-    )
-    (property "Footprint" "Package_TO_SOT_SMD:SOT-23-6" (id 2) (at 238.76 113.03 0)
+    (property "Value" "" (id 1) (at 262.7376 114.173 90)
+      (effects (font (size 1.27 1.27)) (justify left))
+    )
+    (property "Footprint" "" (id 2) (at 238.76 113.03 0)
       (effects (font (size 1.27 1.27)) hide)
     )
     (property "Datasheet" "https://www.st.com/resource/en/datasheet/usblc6-2.pdf" (id 3) (at 260.35 118.11 0)
+      (effects (font (size 1.27 1.27)) hide)
+    )
+    (property "Manufacturer" "ST" (id 4) (at 251.46 113.03 0)
+      (effects (font (size 1.27 1.27)) hide)
+    )
+    (property "Manufacturer Part Number" "USBLC6-2SC6" (id 5) (at 251.46 113.03 0)
+      (effects (font (size 1.27 1.27)) hide)
+    )
+    (property "Supplier" "Digikey" (id 6) (at 251.46 113.03 0)
+      (effects (font (size 1.27 1.27)) hide)
+    )
+    (property "Supplier Part Number" "497-5235-1-ND" (id 7) (at 251.46 113.03 0)
       (effects (font (size 1.27 1.27)) hide)
     )
@@
       (effects (font (size 1.27 1.27)) (justify left))
     )
-    (property "Value" "0.10uF" (id 1) (at 79.121 65.913 0)
-      (effects (font (size 1.27 1.27)) (justify left))
-    )
-    (property "Footprint" "mta1:CAPC1005X06L" (id 2) (at 77.1652 68.58 0)
+    (property "Value" "" (id 1) (at 79.121 65.913 0)
+      (effects (font (size 1.27 1.27)) (justify left))
+    )
+    (property "Footprint" "" (id 2) (at 77.1652 68.58 0)
       (effects (font (size 1.27 1.27)) hide)
     )
     (property "Datasheet" "~" (id 3) (at 76.2 64.77 0)
+      (effects (font (size 1.27 1.27)) hide)
+    )
+    (property "Manufacturer" "Any/not critical" (id 4) (at 76.2 64.77 0)
+      (effects (font (size 1.27 1.27)) hide)
+    )
+    (property "Extended Value" "16V,X5R,20%" (id 5) (at 76.2 64.77 0)
       (effects (font (size 1.27 1.27)) hide)
     )
@@
   )
   (symbol (lib_id "Connector:TestPoint") (at 45.72 60.96 0) (unit 1)
-    (in_bom yes) (on_board yes)
+    (in_bom no) (on_board yes)
     (property "Reference" "TP7" (id 0) (at 47.1932 57.9628 0)
       (effects (font (size 1.27 1.27)) (justify left))
     )
-    (property "Value" "INT_ICE_SCK" (id 1) (at 47.1932 60.2742 0)
-      (effects (font (size 1.27 1.27)) (justify left))
-    )
-    (property "Footprint" "TestPoint:TestPoint_Pad_D1.0mm" (id 2) (at 50.8 60.96 0)
+    (property "Value" "" (id 1) (at 47.1932 60.2742 0)
+      (effects (font (size 1.27 1.27)) (justify left))
+    )
+    (property "Footprint" "" (id 2) (at 50.8 60.96 0)
       (effects (font (size 1.27 1.27)) hide)
     )
@@
   )
   (symbol (lib_id "Connector:TestPoint") (at 45.72 68.58 0) (unit 1)
-    (in_bom yes) (on_board yes)
+    (in_bom no) (on_board yes)
     (property "Reference" "TP8" (id 0) (at 47.1932 65.5828 0)
       (effects (font (size 1.27 1.27)) (justify left))
     )
-    (property "Value" "INT_ICE_SCK" (id 1) (at 47.1932 67.8942 0)
-      (effects (font (size 1.27 1.27)) (justify left))
-    )
-    (property "Footprint" "TestPoint:TestPoint_Pad_D1.0mm" (id 2) (at 50.8 68.58 0)
+    (property "Value" "" (id 1) (at 47.1932 67.8942 0)
+      (effects (font (size 1.27 1.27)) (justify left))
+    )
+    (property "Footprint" "" (id 2) (at 50.8 68.58 0)
       (effects (font (size 1.27 1.27)) hide)
     )
@@
       (effects (font (size 1.27 1.27)) (justify left))
     )
-    (property "Value" "0.10uF" (id 1) (at 79.121 86.233 0)
-      (effects (font (size 1.27 1.27)) (justify left))
-    )
-    (property "Footprint" "mta1:CAPC1005X06L" (id 2) (at 77.1652 88.9 0)
+    (property "Value" "" (id 1) (at 79.121 86.233 0)
+      (effects (font (size 1.27 1.27)) (justify left))
+    )
+    (property "Footprint" "" (id 2) (at 77.1652 88.9 0)
       (effects (font (size 1.27 1.27)) hide)
     )
     (property "Datasheet" "~" (id 3) (at 76.2 85.09 0)
+      (effects (font (size 1.27 1.27)) hide)
+    )
+    (property "Manufacturer" "Any/not critical" (id 4) (at 76.2 85.09 0)
+      (effects (font (size 1.27 1.27)) hide)
+    )
+    (property "Extended Value" "16V,X5R,20%" (id 5) (at 76.2 85.09 0)
       (effects (font (size 1.27 1.27)) hide)
     )
@@
     (in_bom yes) (on_board yes) (fields_autoplaced)
     (property "Reference" "P1" (id 0) (at 190.5 49.53 0))
-    (property "Value" "USB_C_Plug" (id 1) (at 190.5 52.07 0))
-    (property "Footprint" "mta1:U261-241N-4BS60" (id 2) (at 194.31 82.55 0)
+    (property "Value" "" (id 1) (at 190.5 52.07 0))
+    (property "Footprint" "" (id 2) (at 194.31 82.55 0)
       (effects (font (size 1.27 1.27)) hide)
     )
     (property "Datasheet" "https://www.usb.org/sites/default/files/documents/usb_type-c.zip" (id 3) (at 194.31 82.55 0)
+      (effects (font (size 1.27 1.27)) hide)
+    )
+    (property "Manufacturer" "XKB" (id 4) (at 190.5 82.55 0)
+      (effects (font (size 1.27 1.27)) hide)
+    )
+    (property "Manufacturer Part Number" "U261-241N-4BS60" (id 5) (at 190.5 82.55 0)
+      (effects (font (size 1.27 1.27)) hide)
+    )
+    (property "Supplier" "LCSC" (id 6) (at 190.5 82.55 0)
+      (effects (font (size 1.27 1.27)) hide)
+    )
+    (property "Supplier Part Number" "C319150" (id 7) (at 190.5 82.55 0)
       (effects (font (size 1.27 1.27)) hide)
     )
@@
       (effects (font (size 1.27 1.27)) (justify left))
     )
-    (property "Value" "5.1K" (id 1) (at 241.808 72.263 0)
-      (effects (font (size 1.27 1.27)) (justify left))
-    )
-    (property "Footprint" "mta1:ERJ2G(0402)_L" (id 2) (at 238.252 71.12 90)
+    (property "Value" "" (id 1) (at 241.808 72.263 0)
+      (effects (font (size 1.27 1.27)) (justify left))
+    )
+    (property "Footprint" "" (id 2) (at 238.252 71.12 90)
       (effects (font (size 1.27 1.27)) hide)
     )
     (property "Datasheet" "~" (id 3) (at 240.03 71.12 0)
+      (effects (font (size 1.27 1.27)) hide)
+    )
+    (property "Manufacturer" "Any/not critical" (id 4) (at 240.03 71.12 0)
+      (effects (font (size 1.27 1.27)) hide)
+    )
+    (property "Extended Value" "1/16W,1%" (id 5) (at 240.03 71.12 0)
       (effects (font (size 1.27 1.27)) hide)
     )
@@
     (in_bom yes) (on_board yes)
     (property "Reference" "U3" (id 0) (at 106.68 85.09 0))
-    (property "Value" "CH552E" (id 1) (at 123.19 85.09 0))
-    (property "Footprint" "Package_SO:MSOP-10_3x3mm_P0.5mm" (id 2) (at 172.72 107.95 0)
+    (property "Value" "" (id 1) (at 123.19 85.09 0))
+    (property "Footprint" "" (id 2) (at 172.72 107.95 0)
       (effects (font (size 1.27 1.27)) hide)
     )
     (property "Datasheet" "" (id 3) (at 172.72 107.95 0)
+      (effects (font (size 1.27 1.27)) hide)
+    )
+    (property "Manufacturer" "WCH" (id 4) (at 114.3 90.17 0)
+      (effects (font (size 1.27 1.27)) hide)
+    )
+    (property "Manufacturer Part Number" "CH552E" (id 5) (at 114.3 90.17 0)
+      (effects (font (size 1.27 1.27)) hide)
+    )
+    (property "Supplier" "LCSC" (id 6) (at 114.3 90.17 0)
+      (effects (font (size 1.27 1.27)) hide)
+    )
+    (property "Supplier Part Number" "C967938" (id 7) (at 114.3 90.17 0)
       (effects (font (size 1.27 1.27)) hide)
     )
@@
   )
   (symbol (lib_id "Connector:TestPoint") (at 45.72 77.47 0) (unit 1)
-    (in_bom yes) (on_board yes)
+    (in_bom no) (on_board yes)
     (property "Reference" "TP9" (id 0) (at 47.1932 74.4728 0)
       (effects (font (size 1.27 1.27)) (justify left))
     )
-    (property "Value" "INT_ICE_SCK" (id 1) (at 47.1932 76.7842 0)
-      (effects (font (size 1.27 1.27)) (justify left))
-    )
-    (property "Footprint" "TestPoint:TestPoint_Pad_D1.0mm" (id 2) (at 50.8 77.47 0)
+    (property "Value" "" (id 1) (at 47.1932 76.7842 0)
+      (effects (font (size 1.27 1.27)) (justify left))
+    )
+    (property "Footprint" "" (id 2) (at 50.8 77.47 0)
       (effects (font (size 1.27 1.27)) hide)
     )
@@
   )
   (symbol (lib_id "Connector:TestPoint") (at 45.72 53.34 0) (unit 1)
-    (in_bom yes) (on_board yes)
+    (in_bom no) (on_board yes)
     (property "Reference" "TP6" (id 0) (at 47.1932 50.3428 0)
       (effects (font (size 1.27 1.27)) (justify left))
     )
-    (property "Value" "INT_ICE_SCK" (id 1) (at 47.1932 52.6542 0)
-      (effects (font (size 1.27 1.27)) (justify left))
-    )
-    (property "Footprint" "TestPoint:TestPoint_Pad_D1.0mm" (id 2) (at 50.8 53.34 0)
-      (effects (font (size 1.27 1.27)) hide)
-    )
+    (property "Value" "" (id 1) (at 47.1932 52.6542 0)
+      (effects (font (size 1.27 1.27)) (justify left))
+    )
+    (property "Footprint" "" (id 2) (at 50.8 53.34 0)
+      (effects (font (size 1.27 1.27)) hide)
+    )
