File: hw/boards/mta1-usb-v1/mta1-usb-v1.kicad_pcb (KiCad board)
At the start: 4 copper layers, 27.5 x 13.5 mm, 68 parts, among them P1 USB_C_Plug, U1 MCP1824T-2502EOT, U10 PT2043AT6, U2 MIC5258-1.2YM5, U3 CH552E, U5 USBLC6-2SC6, U6 ICE40UP5K-SG48ITR, U8 W25Q80DVUXIE, U9 NCP752BSN33T1G

Commit message: Add extended values, manufacturer/distributor info to components in mta1
Parts:
- C27: value 3pF -> 10pF
- C8: value 10uF 16V -> 10uF
- D1: value Power LED -> 0402 indicator LED, blue
- R16, R17, R18: value 1K -> 1k
- R29: value 5.1K -> 5.1k
- R30: value 2K -> 2k
- TP6: value INT_ICE_SCK -> INT_TX
- TP7: value INT_ICE_SCK -> INT_RX
- TP8: value INT_ICE_SCK -> INT_RTS
- TP9: value INT_ICE_SCK -> INT_CTS
- U8: value W25Q80DVUXIE -> XT25F08BDFIGT-S

Commit message: Update MTA1-USB-V1 release files to match production
* Change SPI flash memory type to XT25F08BDFIGT-S
* Change touch sensor feedback cap to 1uF
* Add manufacturer, manufacturer part number, distributor, distributor part number
Parts:
- C27: value 10pF -> 2.7pF
Changed lines of the file:
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@@
       (effects (font (size 1 1) (thickness 0.15)))
     )
-    (fp_text value "10pF" (at 0 1.16) (layer "F.Fab") hide
+    (fp_text value "2.7pF" (at 0 1.16) (layer "F.Fab") hide
       (effects (font (size 1 1) (thickness 0.15)))
     )
@@
     (descr "Capacitor SMD 1206 (3216 Metric), square (rectangular) end terminal, IPC_7351 nominal, (Body size source: IPC-SM-782 page 76, https://www.pcb-3d.com/wordpress/wp-content/uploads/ipc-sm-782a_amendment_1_and_2.pdf), generated with kicad-footprint-generator")
     (tags "capacitor")
-    (property "Extended Value" "16V")
+    (property "Extended Value" "16V,X5R,10%")
+    (property "Manufacturer" "Fenghua")
+    (property "Manufacturer Part Number" "1206X106K160NT")
     (property "Sheetfile" "application_fpga.kicad_sch")
     (property "Sheetname" "Application FPGA")
+    (property "Supplier" "LCSC")
+    (property "Supplier Part Number" "C105478")
     (attr smd)
     (fp_text reference "C8" (at 3.7 0.2 90) (layer "F.SilkS") hide
