File: hw/boards/mta1-usb-v1/mta1-usb-v1.kicad_pcb (KiCad board)
At the start: 4 copper layers, 27.5 x 13.5 mm, 68 parts, among them P1 USB_C_Plug, U1 MCP1824T-2502EOT, U10 PT2043AT6, U2 MIC5258-1.2YM5, U3 CH552E, U5 USBLC6-2SC6, U6 ICE40UP5K-SG48ITR, U8 W25Q80DVUXIE, U9 NCP752BSN33T1G

Commit message: TK-1 and TP-1 PCBs (#52)
* Add kicad library for flat programming clip

* Add descriptions to part symbols

* Add extended values, manufacturer/distributor info to components in mta1

* Add new board entry for TK1

* Add TP1 programmer design

* Update MTA1-USB-V1 release files to match production

* Change SPI flash memory type to XT25F08BDFIGT-S
* Change touch sensor feedback cap to 1uF
* Add manufacturer, manufacturer part number, distributor, distributor part number

* Update component values for TK1 PCB

* Use specific part # for C8
* Change flash back to Winbond part, for easier sourcing
* Change C1 to 1pF

* Fixes for production programmer PCB

* Swap GND and 5V on J3
* Replace graphic logo with text
* Rename part to 'TP-1'

* TK-1 release

* Add dimensions for PCB
* Add layer stackup for PCB
* Change PCB component origin to match expanded board
* Change schematic title to 'TK-1', update release date

* mta1-usb-v1-programmer: Add corrected part numbers for OSFC production

* Q1, Q2, F1 part subsititutions
* add mfr/supplier info for all parts

* PCB library: add parts

* Rectangular footprint for TK-1 test pads
* BOM generation script used for TK-1 and TP-1 releases

* TP-1 release

* Schematic: Add manufacturer, supplier information for all parts
* Schematic: Update name and release date
* PCB: Add PCB fabrication information
* PCB: Correct pinouts on silkscreen

* PCB library: add 'screw' and 'foot' symbols

* Screw is a schematic-only part, for including mechanical screws in the
  BOM
* Foot is for self-adhesive rubber mounting feet that can be stuck to
  the bottom of a PCB

* TP-1 release: Add screws, feet to the BOM

* Pico library: Add footprint for RPi Pico w/solder paste

* TP-1 RevA release updates:

* Add fiducials in 3 corners (1mm exposed copper ring w/2mm soldermask opening)
* Add solder paste openings to Raspberry Pi Pico pads

* TK-1: RevA.1 release

* Add two fiducials to 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
Parts:
- C27: value 3pF -> 2.7pF
- C8: value 10uF 16V -> 10uF
- D1: value Power LED -> 0402 indicator LED, blue
- R16, R17, R18: value 1K -> 1k
- R29: value 5.1K -> 5.1k
- R30: value 2K -> 2k
- TP6: value INT_ICE_SCK -> INT_TX
- TP7: value INT_ICE_SCK -> INT_RX
- TP8: value INT_ICE_SCK -> INT_RTS
- TP9: value INT_ICE_SCK -> INT_CTS
- U8: value W25Q80DVUXIE -> XT25F08BDFIGT-S
