File: hw/boards/tk1/usb_to_serial.kicad_sch (KiCad schematic)
At the start: 10 parts, among them P1 USB_C_Plug, U3 CH552E, U5 USBLC6-2SC6

Commit message: Update component values for TK1 PCB
* Use specific part # for C8
* Change flash back to Winbond part, for easier sourcing
* Change C1 to 1pF
Parts:
- C13, C7: value 0.10uF -> (none); footprint mta1:CAPC1005X06L -> (none)
- P1: value USB_C_Plug -> (none); footprint mta1:U261-241N-4BS60 -> (none)
- R29: value 5.1k -> (none); footprint mta1:ERJ2G(0402)_L -> (none)
- TP6: value INT_TX -> (none); footprint TestPoint:TestPoint_Pad_D1.0mm -> (none)
- TP7: value INT_RX -> (none); footprint TestPoint:TestPoint_Pad_D1.0mm -> (none)
- TP8: value INT_RTS -> (none); footprint TestPoint:TestPoint_Pad_D1.0mm -> (none)
- TP9: value INT_CTS -> (none); footprint TestPoint:TestPoint_Pad_D1.0mm -> (none)
- U3: value CH552E -> (none); footprint Package_SO:MSOP-10_3x3mm_P0.5mm -> (none)
- U5: value USBLC6-2SC6 -> (none)
Changed lines of the file:
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@@
       (effects (font (size 1.27 1.27)) (justify left))
     )
-    (property "Value" "USBLC6-2SC6" (id 1) (at 262.7376 114.173 90)
+    (property "Value" "" (id 1) (at 262.7376 114.173 90)
       (effects (font (size 1.27 1.27)) (justify left))
     )
@@
       (effects (font (size 1.27 1.27)) (justify left))
     )
-    (property "Value" "0.10uF" (id 1) (at 79.121 65.913 0)
-      (effects (font (size 1.27 1.27)) (justify left))
-    )
-    (property "Footprint" "mta1:CAPC1005X06L" (id 2) (at 77.1652 68.58 0)
+    (property "Value" "" (id 1) (at 79.121 65.913 0)
+      (effects (font (size 1.27 1.27)) (justify left))
+    )
+    (property "Footprint" "" (id 2) (at 77.1652 68.58 0)
       (effects (font (size 1.27 1.27)) hide)
     )
@@
       (effects (font (size 1.27 1.27)) (justify left))
     )
-    (property "Value" "INT_RX" (id 1) (at 47.1932 60.2742 0)
-      (effects (font (size 1.27 1.27)) (justify left))
-    )
-    (property "Footprint" "TestPoint:TestPoint_Pad_D1.0mm" (id 2) (at 50.8 60.96 0)
+    (property "Value" "" (id 1) (at 47.1932 60.2742 0)
+      (effects (font (size 1.27 1.27)) (justify left))
+    )
+    (property "Footprint" "" (id 2) (at 50.8 60.96 0)
       (effects (font (size 1.27 1.27)) hide)
     )
@@
       (effects (font (size 1.27 1.27)) (justify left))
     )
-    (property "Value" "INT_RTS" (id 1) (at 47.1932 67.8942 0)
-      (effects (font (size 1.27 1.27)) (justify left))
-    )
-    (property "Footprint" "TestPoint:TestPoint_Pad_D1.0mm" (id 2) (at 50.8 68.58 0)
+    (property "Value" "" (id 1) (at 47.1932 67.8942 0)
+      (effects (font (size 1.27 1.27)) (justify left))
+    )
+    (property "Footprint" "" (id 2) (at 50.8 68.58 0)
       (effects (font (size 1.27 1.27)) hide)
     )
@@
       (effects (font (size 1.27 1.27)) (justify left))
     )
-    (property "Value" "0.10uF" (id 1) (at 79.121 86.233 0)
-      (effects (font (size 1.27 1.27)) (justify left))
-    )
-    (property "Footprint" "mta1:CAPC1005X06L" (id 2) (at 77.1652 88.9 0)
+    (property "Value" "" (id 1) (at 79.121 86.233 0)
+      (effects (font (size 1.27 1.27)) (justify left))
+    )
+    (property "Footprint" "" (id 2) (at 77.1652 88.9 0)
       (effects (font (size 1.27 1.27)) hide)
     )
@@
     (in_bom yes) (on_board yes) (fields_autoplaced)
     (property "Reference" "P1" (id 0) (at 190.5 49.53 0))
-    (property "Value" "USB_C_Plug" (id 1) (at 190.5 52.07 0))
-    (property "Footprint" "mta1:U261-241N-4BS60" (id 2) (at 194.31 82.55 0)
+    (property "Value" "" (id 1) (at 190.5 52.07 0))
+    (property "Footprint" "" (id 2) (at 194.31 82.55 0)
       (effects (font (size 1.27 1.27)) hide)
     )
@@
       (effects (font (size 1.27 1.27)) (justify left))
     )
-    (property "Value" "5.1k" (id 1) (at 241.808 72.263 0)
-      (effects (font (size 1.27 1.27)) (justify left))
-    )
-    (property "Footprint" "mta1:ERJ2G(0402)_L" (id 2) (at 238.252 71.12 90)
+    (property "Value" "" (id 1) (at 241.808 72.263 0)
+      (effects (font (size 1.27 1.27)) (justify left))
+    )
+    (property "Footprint" "" (id 2) (at 238.252 71.12 90)
       (effects (font (size 1.27 1.27)) hide)
     )
@@
     (in_bom yes) (on_board yes)
     (property "Reference" "U3" (id 0) (at 106.68 85.09 0))
-    (property "Value" "CH552E" (id 1) (at 123.19 85.09 0))
-    (property "Footprint" "Package_SO:MSOP-10_3x3mm_P0.5mm" (id 2) (at 172.72 107.95 0)
+    (property "Value" "" (id 1) (at 123.19 85.09 0))
+    (property "Footprint" "" (id 2) (at 172.72 107.95 0)
       (effects (font (size 1.27 1.27)) hide)
     )
@@
       (effects (font (size 1.27 1.27)) (justify left))
     )
-    (property "Value" "INT_CTS" (id 1) (at 47.1932 76.7842 0)
-      (effects (font (size 1.27 1.27)) (justify left))
-    )
-    (property "Footprint" "TestPoint:TestPoint_Pad_D1.0mm" (id 2) (at 50.8 77.47 0)
+    (property "Value" "" (id 1) (at 47.1932 76.7842 0)
+      (effects (font (size 1.27 1.27)) (justify left))
+    )
+    (property "Footprint" "" (id 2) (at 50.8 77.47 0)
       (effects (font (size 1.27 1.27)) hide)
     )
@@
       (effects (font (size 1.27 1.27)) (justify left))
     )
-    (property "Value" "INT_TX" (id 1) (at 47.1932 52.6542 0)
-      (effects (font (size 1.27 1.27)) (justify left))
-    )
-    (property "Footprint" "TestPoint:TestPoint_Pad_D1.0mm" (id 2) (at 50.8 53.34 0)
-      (effects (font (size 1.27 1.27)) hide)
-    )
+    (property "Value" "" (id 1) (at 47.1932 52.6542 0)
+      (effects (font (size 1.27 1.27)) (justify left))
+    )
+    (property "Footprint" "" (id 2) (at 50.8 53.34 0)
+      (effects (font (size 1.27 1.27)) hide)
+    )

Commit message: TK-1 release
* Add dimensions for PCB
* Add layer stackup for PCB
* Change PCB component origin to match expanded board
* Change schematic title to 'TK-1', update release date
Parts:
- C13, C7: value (none) -> 0.10uF; footprint (none) -> mta1:CAPC1005X06L
- P1: value (none) -> USB_C_Plug; footprint (none) -> mta1:U261-241N-4BS60
- R29: value (none) -> 5.1k; footprint (none) -> mta1:ERJ2G(0402)_L
- TP6: value (none) -> INT_TX; footprint (none) -> mta1:TestPoint_Pad_D1.0mm
- TP7: value (none) -> INT_RX; footprint (none) -> mta1:TestPoint_Pad_D1.0mm
- TP8: value (none) -> INT_RTS; footprint (none) -> mta1:TestPoint_Pad_D1.0mm
- TP9: value (none) -> INT_CTS; footprint (none) -> mta1:TestPoint_Pad_D1.0mm
- U3: value (none) -> CH552E; footprint (none) -> Package_SO:MSOP-10_3x3mm_P0.5mm
- U5: value (none) -> USBLC6-2SC6
Changed lines of the file:
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@@
   (title_block
     (title "USB-to-Serial Interface")
-    (date "2021-09-29")
+    (date "2021-11-14")
     (rev "V1")
     (company "Tillitis AB")
@@
       (effects (font (size 1.27 1.27)) (justify left))
     )
-    (property "Value" "" (id 1) (at 262.7376 114.173 90)
+    (property "Value" "USBLC6-2SC6" (id 1) (at 262.7376 114.173 90)
       (effects (font (size 1.27 1.27)) (justify left))
     )
@@
       (effects (font (size 1.27 1.27)) (justify left))
     )
-    (property "Value" "" (id 1) (at 79.121 65.913 0)
-      (effects (font (size 1.27 1.27)) (justify left))
-    )
-    (property "Footprint" "" (id 2) (at 77.1652 68.58 0)
+    (property "Value" "0.10uF" (id 1) (at 79.121 65.913 0)
+      (effects (font (size 1.27 1.27)) (justify left))
+    )
+    (property "Footprint" "mta1:CAPC1005X06L" (id 2) (at 77.1652 68.58 0)
       (effects (font (size 1.27 1.27)) hide)
     )
@@
       (effects (font (size 1.27 1.27)) (justify left))
     )
-    (property "Value" "" (id 1) (at 47.1932 60.2742 0)
-      (effects (font (size 1.27 1.27)) (justify left))
-    )
-    (property "Footprint" "" (id 2) (at 50.8 60.96 0)
+    (property "Value" "INT_RX" (id 1) (at 47.1932 60.2742 0)
+      (effects (font (size 1.27 1.27)) (justify left))
+    )
+    (property "Footprint" "mta1:TestPoint_Pad_D1.0mm" (id 2) (at 50.8 60.96 0)
       (effects (font (size 1.27 1.27)) hide)
     )
@@
       (effects (font (size 1.27 1.27)) (justify left))
     )
-    (property "Value" "" (id 1) (at 47.1932 67.8942 0)
-      (effects (font (size 1.27 1.27)) (justify left))
-    )
-    (property "Footprint" "" (id 2) (at 50.8 68.58 0)
+    (property "Value" "INT_RTS" (id 1) (at 47.1932 67.8942 0)
+      (effects (font (size 1.27 1.27)) (justify left))
+    )
+    (property "Footprint" "mta1:TestPoint_Pad_D1.0mm" (id 2) (at 50.8 68.58 0)
       (effects (font (size 1.27 1.27)) hide)
     )
@@
       (effects (font (size 1.27 1.27)) (justify left))
     )
-    (property "Value" "" (id 1) (at 79.121 86.233 0)
-      (effects (font (size 1.27 1.27)) (justify left))
-    )
-    (property "Footprint" "" (id 2) (at 77.1652 88.9 0)
+    (property "Value" "0.10uF" (id 1) (at 79.121 86.233 0)
+      (effects (font (size 1.27 1.27)) (justify left))
+    )
+    (property "Footprint" "mta1:CAPC1005X06L" (id 2) (at 77.1652 88.9 0)
       (effects (font (size 1.27 1.27)) hide)
     )
@@
     (in_bom yes) (on_board yes) (fields_autoplaced)
     (property "Reference" "P1" (id 0) (at 190.5 49.53 0))
-    (property "Value" "" (id 1) (at 190.5 52.07 0))
-    (property "Footprint" "" (id 2) (at 194.31 82.55 0)
+    (property "Value" "USB_C_Plug" (id 1) (at 190.5 52.07 0))
+    (property "Footprint" "mta1:U261-241N-4BS60" (id 2) (at 194.31 82.55 0)
       (effects (font (size 1.27 1.27)) hide)
     )
@@
       (effects (font (size 1.27 1.27)) (justify left))
     )
-    (property "Value" "" (id 1) (at 241.808 72.263 0)
-      (effects (font (size 1.27 1.27)) (justify left))
-    )
-    (property "Footprint" "" (id 2) (at 238.252 71.12 90)
+    (property "Value" "5.1k" (id 1) (at 241.808 72.263 0)
+      (effects (font (size 1.27 1.27)) (justify left))
+    )
+    (property "Footprint" "mta1:ERJ2G(0402)_L" (id 2) (at 238.252 71.12 90)
       (effects (font (size 1.27 1.27)) hide)
     )
@@
     (in_bom yes) (on_board yes)
     (property "Reference" "U3" (id 0) (at 106.68 85.09 0))
-    (property "Value" "" (id 1) (at 123.19 85.09 0))
-    (property "Footprint" "" (id 2) (at 172.72 107.95 0)
+    (property "Value" "CH552E" (id 1) (at 123.19 85.09 0))
+    (property "Footprint" "Package_SO:MSOP-10_3x3mm_P0.5mm" (id 2) (at 172.72 107.95 0)
       (effects (font (size 1.27 1.27)) hide)
     )
@@
       (effects (font (size 1.27 1.27)) (justify left))
     )
-    (property "Value" "" (id 1) (at 47.1932 76.7842 0)
-      (effects (font (size 1.27 1.27)) (justify left))
-    )
-    (property "Footprint" "" (id 2) (at 50.8 77.47 0)
+    (property "Value" "INT_CTS" (id 1) (at 47.1932 76.7842 0)
+      (effects (font (size 1.27 1.27)) (justify left))
+    )
+    (property "Footprint" "mta1:TestPoint_Pad_D1.0mm" (id 2) (at 50.8 77.47 0)
       (effects (font (size 1.27 1.27)) hide)
     )
@@
       (effects (font (size 1.27 1.27)) (justify left))
     )
-    (property "Value" "" (id 1) (at 47.1932 52.6542 0)
-      (effects (font (size 1.27 1.27)) (justify left))
-    )
-    (property "Footprint" "" (id 2) (at 50.8 53.34 0)
-      (effects (font (size 1.27 1.27)) hide)
-    )
+    (property "Value" "INT_TX" (id 1) (at 47.1932 52.6542 0)
+      (effects (font (size 1.27 1.27)) (justify left))
+    )
+    (property "Footprint" "mta1:TestPoint_Pad_D1.0mm" (id 2) (at 50.8 53.34 0)
+      (effects (font (size 1.27 1.27)) hide)
+    )
