File: hw/boards/tk1/powersupply.kicad_sch (KiCad schematic)
At the start: 19 parts

Commit message: TK-1 release
* Add dimensions for PCB
* Add layer stackup for PCB
* Change PCB component origin to match expanded board
* Change schematic title to 'TK-1', update release date
Parts:
- C1, C2, C3, C4, C5, C6: value (none) -> 10uF; footprint (none) -> mta1:CAPC1608X09L
- D1: value (none) -> 0402 indicator LED, blue; footprint (none) -> LED_SMD:LED_0402_1005Metric
- R1, R2, R22: value (none) -> 10k; footprint (none) -> mta1:ERJ2G(0402)_L
- R3: value (none) -> 1k; footprint (none) -> mta1:ERJ2G(0402)_L
- TP1: value (none) -> 5V; footprint (none) -> mta1:TestPoint_Pad_D1.0mm
- TP2: value (none) -> 3V3; footprint (none) -> mta1:TestPoint_Pad_D1.0mm
- TP28: value (none) -> GND; footprint (none) -> mta1:TestPoint_Pad_D1.0mm
- TP3: value (none) -> 2V5; footprint (none) -> mta1:TestPoint_Pad_D1.0mm
- TP4: value (none) -> 1V2; footprint (none) -> mta1:TestPoint_Pad_D1.0mm
- U1: value (none) -> MCP1824T-2502EOT
- U2: value (none) -> MIC5258-1.2YM5
- U9: value (none) -> NCP752BSN33T1G; footprint (none) -> mta1:NCP752BSN33T1G
Changed lines of the file:
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@@
   (title_block
     (title "Power Supply")
-    (date "2021-09-29")
+    (date "2021-11-14")
     (rev "V1")
     (company "Tillitis AB")
@@
       (effects (font (size 1.27 1.27)) (justify left))
     )
-    (property "Value" "" (id 1) (at 33.401 39.243 0)
+    (property "Value" "10uF" (id 1) (at 33.401 39.243 0)
       (effects (font (size 1.27 1.27)) (justify left))
     )
-    (property "Footprint" "" (id 2) (at 31.4452 41.91 0)
+    (property "Footprint" "mta1:CAPC1608X09L" (id 2) (at 31.4452 41.91 0)
       (effects (font (size 1.27 1.27)) hide)
     )
@@
       (effects (font (size 1.27 1.27)) (justify left))
     )
-    (property "Value" "" (id 1) (at 43.688 39.243 0)
+    (property "Value" "10k" (id 1) (at 43.688 39.243 0)
       (effects (font (size 1.27 1.27)) (justify left))
     )
-    (property "Footprint" "" (id 2) (at 40.132 38.1 90)
+    (property "Footprint" "mta1:ERJ2G(0402)_L" (id 2) (at 40.132 38.1 90)
       (effects (font (size 1.27 1.27)) hide)
     )
@@
       (effects (font (size 1.27 1.27)) (justify left))
     )
-    (property "Value" "" (id 1) (at 98.171 49.403 0)
+    (property "Value" "10uF" (id 1) (at 98.171 49.403 0)
       (effects (font (size 1.27 1.27)) (justify left))
     )
-    (property "Footprint" "" (id 2) (at 96.2152 52.07 0)
+    (property "Footprint" "mta1:CAPC1608X09L" (id 2) (at 96.2152 52.07 0)
       (effects (font (size 1.27 1.27)) hide)
     )
@@
       (effects (font (size 1.27 1.27)) (justify left))
     )
-    (property "Value" "" (id 1) (at 88.138 57.023 0)
+    (property "Value" "10k" (id 1) (at 88.138 57.023 0)
       (effects (font (size 1.27 1.27)) (justify left))
     )
-    (property "Footprint" "" (id 2) (at 84.582 55.88 90)
+    (property "Footprint" "mta1:ERJ2G(0402)_L" (id 2) (at 84.582 55.88 90)
       (effects (font (size 1.27 1.27)) hide)
     )
@@
       (effects (font (size 1.27 1.27)) (justify left))
     )
-    (property "Value" "" (id 1) (at 100.711 97.663 0)
+    (property "Value" "10uF" (id 1) (at 100.711 97.663 0)
       (effects (font (size 1.27 1.27)) (justify left))
     )
-    (property "Footprint" "" (id 2) (at 98.7552 100.33 0)
+    (property "Footprint" "mta1:CAPC1608X09L" (id 2) (at 98.7552 100.33 0)
       (effects (font (size 1.27 1.27)) hide)
     )
@@
     (in_bom yes) (on_board yes)
     (property "Reference" "U2" (id 0) (at 64.77 35.56 0))
-    (property "Value" "" (id 1) (at 64.77 38.1 0))
+    (property "Value" "MIC5258-1.2YM5" (id 1) (at 64.77 38.1 0))
     (property "Footprint" "Package_TO_SOT_SMD:SOT-23-5" (id 2) (at 64.77 34.29 0)
       (effects (font (size 1.27 1.27)) hide)
@@
     (in_bom yes) (on_board yes)
     (property "Reference" "U1" (id 0) (at 64.77 135.89 0))
-    (property "Value" "" (id 1) (at 64.77 138.43 0))
+    (property "Value" "MCP1824T-2502EOT" (id 1) (at 64.77 138.43 0))
     (property "Footprint" "Package_TO_SOT_SMD:SOT-23-5" (id 2) (at 83.82 156.21 0)
       (effects (font (size 1.27 1.27)) hide)
@@
       (effects (font (size 1.27 1.27)) (justify left))
     )
-    (property "Value" "" (id 1) (at 30.861 152.273 0)
+    (property "Value" "10uF" (id 1) (at 30.861 152.273 0)
       (effects (font (size 1.27 1.27)) (justify left))
     )
-    (property "Footprint" "" (id 2) (at 28.9052 154.94 0)
+    (property "Footprint" "mta1:CAPC1608X09L" (id 2) (at 28.9052 154.94 0)
       (effects (font (size 1.27 1.27)) hide)
     )
@@
       (effects (font (size 1.27 1.27)) (justify left))
     )
-    (property "Value" "" (id 1) (at 95.631 152.273 0)
+    (property "Value" "10uF" (id 1) (at 95.631 152.273 0)
       (effects (font (size 1.27 1.27)) (justify left))
     )
-    (property "Footprint" "" (id 2) (at 93.6752 154.94 0)
+    (property "Footprint" "mta1:CAPC1608X09L" (id 2) (at 93.6752 154.94 0)
       (effects (font (size 1.27 1.27)) hide)
     )
@@
       (effects (font (size 1.27 1.27)) (justify left))
     )
-    (property "Value" "" (id 1) (at 136.0932 100.9142 0)
+    (property "Value" "3V3" (id 1) (at 136.0932 100.9142 0)
       (effects (font (size 1.27 1.27)) (justify left))
     )
-    (property "Footprint" "" (id 2) (at 139.7 101.6 0)
+    (property "Footprint" "mta1:TestPoint_Pad_D1.0mm" (id 2) (at 139.7 101.6 0)
       (effects (font (size 1.27 1.27)) hide)
     )
@@
       (effects (font (size 1.27 1.27)) (justify left))
     )
-    (property "Value" "" (id 1) (at 148.59 100.33 0)
+    (property "Value" "2V5" (id 1) (at 148.59 100.33 0)
       (effects (font (size 1.27 1.27)) (justify left))
     )
-    (property "Footprint" "" (id 2) (at 152.4 101.6 0)
+    (property "Footprint" "mta1:TestPoint_Pad_D1.0mm" (id 2) (at 152.4 101.6 0)
       (effects (font (size 1.27 1.27)) hide)
     )
@@
       (effects (font (size 1.27 1.27)) (justify left))
     )
-    (property "Value" "" (id 1) (at 164.0332 100.9142 0)
+    (property "Value" "1V2" (id 1) (at 164.0332 100.9142 0)
       (effects (font (size 1.27 1.27)) (justify left))
     )
-    (property "Footprint" "" (id 2) (at 167.64 101.6 0)
+    (property "Footprint" "mta1:TestPoint_Pad_D1.0mm" (id 2) (at 167.64 101.6 0)
       (effects (font (size 1.27 1.27)) hide)
     )
@@
     (in_bom yes) (on_board yes)
     (property "Reference" "U9" (id 0) (at 63.5 83.3882 0))
-    (property "Value" "" (id 1) (at 63.5 85.6996 0))
-    (property "Footprint" "" (id 2) (at 63.5 83.82 0)
+    (property "Value" "NCP752BSN33T1G" (id 1) (at 63.5 85.6996 0))
+    (property "Footprint" "mta1:NCP752BSN33T1G" (id 2) (at 63.5 83.82 0)
       (effects (font (size 1.27 1.27)) hide)
     )
@@
       (effects (font (size 1.27 1.27)) (justify left))
     )
-    (property "Value" "" (id 1) (at 35.941 98.933 0)
+    (property "Value" "10uF" (id 1) (at 35.941 98.933 0)
       (effects (font (size 1.27 1.27)) (justify left))
     )
-    (property "Footprint" "" (id 2) (at 33.9852 101.6 0)
+    (property "Footprint" "mta1:CAPC1608X09L" (id 2) (at 33.9852 101.6 0)
       (effects (font (size 1.27 1.27)) hide)
     )
@@
       (effects (font (size 1.27 1.27)) (justify left))
     )
-    (property "Value" "" (id 1) (at 142.748 154.813 0)
+    (property "Value" "1k" (id 1) (at 142.748 154.813 0)
       (effects (font (size 1.27 1.27)) (justify left))
     )
-    (property "Footprint" "" (id 2) (at 139.192 153.67 90)
+    (property "Footprint" "mta1:ERJ2G(0402)_L" (id 2) (at 139.192 153.67 90)
       (effects (font (size 1.27 1.27)) hide)
     )
@@
       (effects (font (size 1.27 1.27)) (justify right))
     )
-    (property "Value" "" (id 1) (at 143.9672 146.1008 90)
+    (property "Value" "0402 indicator LED, blue" (id 1) (at 143.9672 146.1008 90)
       (effects (font (size 1.27 1.27)) (justify right))
     )
-    (property "Footprint" "" (id 2) (at 140.97 144.78 0)
+    (property "Footprint" "LED_SMD:LED_0402_1005Metric" (id 2) (at 140.97 144.78 0)
       (effects (font (size 1.27 1.27)) hide)
     )
@@
       (effects (font (size 1.27 1.27)) (justify left))
     )
-    (property "Value" "" (id 1) (at 123.3932 100.9142 0)
+    (property "Value" "5V" (id 1) (at 123.3932 100.9142 0)
       (effects (font (size 1.27 1.27)) (justify left))
     )
-    (property "Footprint" "" (id 2) (at 127 101.6 0)
+    (property "Footprint" "mta1:TestPoint_Pad_D1.0mm" (id 2) (at 127 101.6 0)
       (effects (font (size 1.27 1.27)) hide)
     )
@@
       (effects (font (size 1.27 1.27)) (justify left))
     )
-    (property "Value" "" (id 1) (at 86.868 105.283 0)
+    (property "Value" "10k" (id 1) (at 86.868 105.283 0)
       (effects (font (size 1.27 1.27)) (justify left))
     )
-    (property "Footprint" "" (id 2) (at 83.312 104.14 90)
+    (property "Footprint" "mta1:ERJ2G(0402)_L" (id 2) (at 83.312 104.14 90)
       (effects (font (size 1.27 1.27)) hide)
     )
@@
       (effects (font (size 1.27 1.27)) (justify left))
     )
-    (property "Value" "" (id 1) (at 164.0332 113.6142 0)
+    (property "Value" "GND" (id 1) (at 164.0332 113.6142 0)
       (effects (font (size 1.27 1.27)) (justify left))
     )
-    (property "Footprint" "" (id 2) (at 167.64 114.3 0)
+    (property "Footprint" "mta1:TestPoint_Pad_D1.0mm" (id 2) (at 167.64 114.3 0)
       (effects (font (size 1.27 1.27)) hide)
     )
