File: hw/boards/tp1/tp1.kicad_pcb (KiCad board)
At the start: 2 copper layers, 45 x 87 mm, 20 parts, among them J1 Conn_01x20, J2 Conn_01x20, J3 BC-1-208, J4 BC-1-701, Q1 AO3400A, Q2 AO3401A, U2 Pico

Commit message: Fixes for production programmer PCB
* Swap GND and 5V on J3
* Replace graphic logo with text
* Rename part to 'TP-1'
Parts:
- removed G***: LOGO, mta1:tillitis_logo
- F1: value 50mA, nSMD005 -> 50mA
Connections:
- J3 pad 1: GND -> /5V_DUT
- J3 pad 2: /5V_DUT -> GND
Routing:
- net /5V_DUT: track 30.3 -> 29.5 mm
Other:
- board text added: "TK-1 PINS"
- board text added: "TP-1 RevA 2022-11"
- board text added: "Tillitis TK-1 Programmer"
- board text added: "Tillitis TK-1 Programmer TP-1 RevA"
- board text removed: "+1V2"
- board text removed: "+2V5"
- board text removed: "+3V3"
- board text removed: "Programmer RevA 2022-11"
- board text removed: "TK1 PINS"
- board text removed: "Tillitis Key Programmer RevA"

Commit message: TP-1 release
* Schematic: Add manufacturer, supplier information for all parts
* Schematic: Update name and release date
* PCB: Add PCB fabrication information
* PCB: Correct pinouts on silkscreen
Routing:
- net /5V_FUSE: track 125.1 -> 121.9 mm
Other:
- board text added: "0.2000 mm / 0.0000 mm"
- board text added: "0.3000 mm"
- board text added: "1.6000 mm"
- board text added: "2"
- board text added: "45.0000 mm x 86.9929 mm"
- board text added: "ADC1"
- board text added: "BOARD CHARACTERISTICS"
- board text added: "Board Thickness:"
- board text added: "Board overall dimensions:"
- board text added: "Castellated pads:"
- board text added: "Copper Finish:"
- board text added: "Copper Layer Count:"
- board text added: "ENIG"
- board text added: "Edge card connectors:"
- board text added: "Impedance Control:"
- board text added: "Min hole diameter:"
- board text added: "Min track/spacing:"
- board text added: "No"
- board text added: "Plated Board Edge:"

Commit message: TP-1 release: Add screws, feet to the BOM
Parts:
- R11, R12, R13, R14, R15, R16, R17: value R100 -> 100R
Changed lines of the file:
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@@
       (effects (font (size 1 1) (thickness 0.15)))
     )
-    (fp_text value "R100" (at 0 1.17 90) (layer "F.Fab")
+    (fp_text value "100R" (at 0 1.17 90) (layer "F.Fab")
       (effects (font (size 1 1) (thickness 0.15)))
     )
@@
       (effects (font (size 1 1) (thickness 0.15)))
     )
-    (fp_text value "R100" (at 0 1.17 90) (layer "F.Fab")
+    (fp_text value "100R" (at 0 1.17 90) (layer "F.Fab")
       (effects (font (size 1 1) (thickness 0.15)))
     )
@@
       (effects (font (size 1 1) (thickness 0.15)))
     )
-    (fp_text value "R100" (at 0 1.17 90) (layer "F.Fab")
+    (fp_text value "100R" (at 0 1.17 90) (layer "F.Fab")
       (effects (font (size 1 1) (thickness 0.15)))
     )
@@
       (effects (font (size 1 1) (thickness 0.15)))
     )
-    (fp_text value "R100" (at 0 1.17 90) (layer "F.Fab")
+    (fp_text value "100R" (at 0 1.17 90) (layer "F.Fab")
       (effects (font (size 1 1) (thickness 0.15)))
     )
@@
       (effects (font (size 1 1) (thickness 0.15)))
     )
-    (fp_text value "R100" (at 0 1.17 90) (layer "F.Fab")
+    (fp_text value "100R" (at 0 1.17 90) (layer "F.Fab")
       (effects (font (size 1 1) (thickness 0.15)))
     )
@@
       (effects (font (size 1 1) (thickness 0.15)))
     )
-    (fp_text value "R100" (at 0 1.17 90) (layer "F.Fab")
+    (fp_text value "100R" (at 0 1.17 90) (layer "F.Fab")
       (effects (font (size 1 1) (thickness 0.15)))
     )
@@
       (effects (font (size 1 1) (thickness 0.15)))
     )
-    (fp_text value "R100" (at 0 1.17 90) (layer "F.Fab")
-      (effects (font (size 1 1) (thickness 0.15)))
-    )
+    (fp_text value "100R" (at 0 1.17 90) (layer "F.Fab")
+      (effects (font (size 1 1) (thickness 0.15)))
+    )

Commit message: TP-1 RevA release updates:
* Add fiducials in 3 corners (1mm exposed copper ring w/2mm soldermask opening)
* Add solder paste openings to Raspberry Pi Pico pads
Parts:
- added FID1: Fiducial, Fiducial:Fiducial_1mm_Mask2mm, F.Cu at (161.0, 134.0)
- added FID2: Fiducial, Fiducial:Fiducial_1mm_Mask2mm, F.Cu at (120.0, 51.0)
- added FID3: Fiducial, Fiducial:Fiducial_1mm_Mask2mm, F.Cu at (120.0, 134.0)
- U2: footprint MCU_RaspberryPi_and_Boards:RPi_Pico_SMD -> MCU_RaspberryPi_and_Boards:RPi_Pico_SMD_reflow

Commit message: Make placement diagrams for TP-1, TK-1
* Update BC-1-xxx footprints to include placement outlines
* Update TP-1 PCB with new footprints, clean up top fab layer
* Take screenshots of top layers of both boards
Parts:
- renumbered FID3 to FIDe
Changed lines of the file:
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@@
       (effects (font (size 1 1) (thickness 0.15)))
     )
-    (fp_text value "Conn_01x20" (at 0 50.59) (layer "F.Fab")
+    (fp_text value "Conn_01x20" (at 0 50.59) (layer "F.Fab") hide
       (effects (font (size 1 1) (thickness 0.15)))
     )
@@
       (effects (font (size 1 1) (thickness 0.15)))
     )
-    (fp_text value "50mA" (at 0 1.82 90) (layer "F.Fab")
+    (fp_text value "50mA" (at 0 1.82 90) (layer "F.Fab") hide
       (effects (font (size 1 1) (thickness 0.15)))
     )
@@
       (effects (font (size 1 1) (thickness 0.15)))
     )
-    (fp_text value "Fiducial" (at 0 2) (layer "F.Fab")
+    (fp_text value "Fiducial" (at 0 2) (layer "F.Fab") hide
       (effects (font (size 1 1) (thickness 0.15)))
     )
@@
       (effects (font (size 1 1) (thickness 0.15)))
     )
-    (fp_text value "100R" (at 0 1.17 90) (layer "F.Fab")
+    (fp_text value "100R" (at 0 1.17 90) (layer "F.Fab") hide
       (effects (font (size 1 1) (thickness 0.15)))
     )
@@
       (effects (font (size 1 1) (thickness 0.15)))
     )
-    (fp_text value "Conn_01x20" (at 0 50.59) (layer "F.Fab")
+    (fp_text value "Conn_01x20" (at 0 50.59) (layer "F.Fab") hide
       (effects (font (size 1 1) (thickness 0.15)))
     )
@@
       (effects (font (size 1 1) (thickness 0.15)))
     )
-    (fp_text value "100R" (at 0 1.17 90) (layer "F.Fab")
+    (fp_text value "100R" (at 0 1.17 90) (layer "F.Fab") hide
       (effects (font (size 1 1) (thickness 0.15)))
     )
@@
       (effects (font (size 1 1) (thickness 0.15)))
     )
-    (fp_text value "100R" (at 0 1.17 90) (layer "F.Fab")
+    (fp_text value "100R" (at 0 1.17 90) (layer "F.Fab") hide
       (effects (font (size 1 1) (thickness 0.15)))
     )
@@
       (effects (font (size 1 1) (thickness 0.15)))
     )
-    (fp_text value "100R" (at 0 1.17 90) (layer "F.Fab")
+    (fp_text value "100R" (at 0 1.17 90) (layer "F.Fab") hide
       (effects (font (size 1 1) (thickness 0.15)))
     )
@@
       (effects (font (size 1 1) (thickness 0.15)))
     )
-    (fp_text value "AO3400A" (at 0 -0.09) (layer "F.Fab")
+    (fp_text value "AO3400A" (at 0 -0.09) (layer "F.Fab") hide
       (effects (font (size 1 1) (thickness 0.15)))
     )
@@
       (effects (font (size 1 1) (thickness 0.15)))
     )
-    (fp_text value "mta1_usb_ch552_flat" (at 2.1 2.5 90 unlocked) (layer "F.Fab")
-      (effects (font (size 1 1) (thickness 0.15)))
-    )
-    (fp_text user "${REFERENCE}" (at 0 0 90 unlocked) (layer "F.Fab")
+    (fp_text value "mta1_usb_ch552_flat" (at 2.1 2.5 90 unlocked) (layer "F.Fab") hide
+      (effects (font (size 1 1) (thickness 0.15)))
+    )
+    (fp_text user "${REFERENCE}" (at -0.142 3.764 90 unlocked) (layer "F.Fab") hide
       (effects (font (size 1 1) (thickness 0.15)))
     )
@@
       (effects (font (size 1 1) (thickness 0.15)))
     )
-    (fp_text value "10K" (at 0 1.17 90) (layer "F.Fab")
+    (fp_text value "10K" (at 0 1.17 90) (layer "F.Fab") hide
       (effects (font (size 1 1) (thickness 0.15)))
     )
@@
       (effects (font (size 1 1) (thickness 0.15)))
     )
-    (fp_text value "AO3401A" (at -0.1 0) (layer "F.Fab")
+    (fp_text value "AO3401A" (at -0.1 0) (layer "F.Fab") hide
       (effects (font (size 1 1) (thickness 0.15)))
     )
@@
       (effects (font (size 1 1) (thickness 0.15)))
     )
-    (fp_text value "BC-1-701" (at 0 9 180 unlocked) (layer "F.Fab")
-      (effects (font (size 1 1) (thickness 0.15)))
-    )
-    (fp_line (start -3 -7) (end 3 -7) (layer "F.SilkS") (width 0.12))
+    (fp_text value "BC-1-701" (at 0 9 180 unlocked) (layer "F.Fab") hide
+      (effects (font (size 1 1) (thickness 0.15)))
+    )
+    (fp_text user "${REFERENCE}" (at 0 0 unlocked) (layer "F.Fab")
+      (effects (font (size 1 1) (thickness 0.15)))
+    )
     (fp_line (start -3 7) (end -3 -7) (layer "F.SilkS") (width 0.12))
     (fp_line (start 3 7) (end -3 7) (layer "F.SilkS") (width 0.12))
+    (fp_line (start -3 -7) (end 3 -7) (layer "F.SilkS") (width 0.12))
+    (fp_line (start -3.5 7.5) (end 3.5 7.5) (layer "F.CrtYd") (width 0.05))
+    (fp_line (start -3.5 -7.5) (end 3.5 -7.5) (layer "F.CrtYd") (width 0.05))
     (fp_line (start -3.5 7.5) (end -3.5 -7.5) (layer "F.CrtYd") (width 0.05))
-    (fp_line (start -3.5 -7.5) (end 3.5 -7.5) (layer "F.CrtYd") (width 0.05))
-    (fp_line (start -3.5 7.5) (end 3.5 7.5) (layer "F.CrtYd") (width 0.05))
     (fp_line (start 3.5 7.5) (end 3.5 -7.5) (layer "F.CrtYd") (width 0.05))
+    (fp_line (start -3 7) (end 3 7) (layer "F.Fab") (width 0.12))
+    (fp_line (start 3 7) (end 3 -7) (layer "F.Fab") (width 0.12))
+    (fp_line (start -3 7) (end -3 -7) (layer "F.Fab") (width 0.12))
+    (fp_line (start -3 -7) (end 3 -7) (layer "F.Fab") (width 0.12))
     (pad "1" smd roundrect (at 2 -6 180) (size 2.6 1.7) (layers "F.Cu" "F.Paste" "F.Mask") (roundrect_rratio 0.1)
       (net 11 "/SCK") (pinfunction "1") (pintype "passive"))
@@
       (effects (font (size 1 1) (thickness 0.15)))
     )
-    (fp_text value "BC-1-208" (at 0 3.5 unlocked) (layer "F.Fab")
-      (effects (font (size 1 1) (thickness 0.15)))
-    )
-    (fp_text user "${REFERENCE}" (at -1.95 0.85 unlocked) (layer "F.Fab")
-      (effects (font (size 1 1) (thickness 0.15)))
-    )
+    (fp_text value "BC-1-208" (at 0 3.5 unlocked) (layer "F.Fab") hide
+      (effects (font (size 1 1) (thickness 0.15)))
+    )
+    (fp_text user "${REFERENCE}" (at 0.014 0.322 unlocked) (layer "F.Fab")
+      (effects (font (size 1 1) (thickness 0.15)))
+    )
+    (fp_line (start -3 -2) (end 3 -2) (layer "F.SilkS") (width 0.12))
+    (fp_line (start -3 2) (end -3 -2) (layer "F.SilkS") (width 0.12))
     (fp_line (start 3 2) (end -3 2) (layer "F.SilkS") (width 0.12))
-    (fp_line (start -3 2) (end -3 -2) (layer "F.SilkS") (width 0.12))
-    (fp_line (start -3 -2) (end 3 -2) (layer "F.SilkS") (width 0.12))
     (fp_line (start -3.5 -2.5) (end 3.5 -2.5) (layer "F.CrtYd") (width 0.05))
-    (fp_line (start 3.5 2.5) (end 3.5 -2.5) (layer "F.CrtYd") (width 0.05))
     (fp_line (start -3.5 2.5) (end 3.5 2.5) (layer "F.CrtYd") (width 0.05))
     (fp_line (start -3.5 2.5) (end -3.5 -2.5) (layer "F.CrtYd") (width 0.05))
+    (fp_line (start 3.5 2.5) (end 3.5 -2.5) (layer "F.CrtYd") (width 0.05))
+    (fp_line (start -3 -2) (end 3 -2) (layer "F.Fab") (width 0.12))
+    (fp_line (start -3 2) (end 3 2) (layer "F.Fab") (width 0.12))
+    (fp_line (start -3 2) (end -3 -2) (layer "F.Fab") (width 0.12))
+    (fp_line (start 3 2) (end 3 -2) (layer "F.Fab") (width 0.12))
     (pad "1" smd roundrect (at 2 -1) (size 2.6 1.7) (layers "F.Cu" "F.Paste" "F.Mask") (roundrect_rratio 0.1)
       (net 43 "/5V_DUT") (pinfunction "1") (pintype "passive"))
@@
       (effects (font (size 1 1) (thickness 0.15)))
     )
-    (fp_text value "Pico" (at 0 2.159) (layer "F.Fab")
+    (fp_text value "Pico" (at 0 2.159) (layer "F.Fab") hide
       (effects (font (size 1 1) (thickness 0.15)))
     )
@@
       (effects (font (size 1 1) (thickness 0.15)))
     )
-    (fp_text value "100R" (at 0 1.17 90) (layer "F.Fab")
+    (fp_text value "100R" (at 0 1.17 90) (layer "F.Fab") hide
       (effects (font (size 1 1) (thickness 0.15)))
     )
@@
     (property "Sheetname" "")
     (attr smd)
-    (fp_text reference "FID3" (at 0 -2) (layer "F.SilkS") hide
-      (effects (font (size 1 1) (thickness 0.15)))
-    )
-    (fp_text value "Fiducial" (at 0 2) (layer "F.Fab")
+    (fp_text reference "FIDe" (at 0 -2) (layer "F.SilkS") hide
+      (effects (font (size 1 1) (thickness 0.15)))
+    )
+    (fp_text value "Fiducial" (at 0 2) (layer "F.Fab") hide
       (effects (font (size 1 1) (thickness 0.15)))
     )
@@
       (effects (font (size 1 1) (thickness 0.15)))
     )
-    (fp_text value "100R" (at 0 1.17 90) (layer "F.Fab")
+    (fp_text value "100R" (at 0 1.17 90) (layer "F.Fab") hide
       (effects (font (size 1 1) (thickness 0.15)))
     )
@@
       (effects (font (size 1 1) (thickness 0.15)))
     )
-    (fp_text value "100R" (at 0 1.17 90) (layer "F.Fab")
+    (fp_text value "100R" (at 0 1.17 90) (layer "F.Fab") hide
       (effects (font (size 1 1) (thickness 0.15)))
     )
@@
       (effects (font (size 1 1) (thickness 0.15)))
     )
-    (fp_text value "10K" (at 0 1.17 -270) (layer "F.Fab")
+    (fp_text value "10K" (at 0 1.17 -270) (layer "F.Fab") hide
       (effects (font (size 1 1) (thickness 0.15)))
     )
@@
       (effects (font (size 1 1) (thickness 0.15)))
     )
-    (fp_text value "Fiducial" (at 0 2) (layer "F.Fab")
-      (effects (font (size 1 1) (thickness 0.15)))
-    )
+    (fp_text value "Fiducial" (at 0 2) (layer "F.Fab") hide
+      (effects (font (size 1 1) (thickness 0.15)))
+    )
